File: PCBs/LED_boards/led_boards.kicad_pcb (KiCad board)
At the start: 2 copper layers, 48.9 x 36.5 mm, 15 parts, among them J1 from_shield, J2 from_shield

Commit message: create PCBs for easier replication of the system. It has been altered to use an arduino Mega, instead of an arduino Uno.
Parts:
- removed D3: LED_RGBK, LED_THT:LED_D5.0mm-4_RGB_Wide_Pins
- removed D4: LED, LED_THT:LED_D5.0mm
- removed J1, J2: from_shield, Connector_IDC:IDC-Header_2x05_P2.54mm_Vertical
- removed R5, R6, R7, R8: 220ohms, Resistor_THT:R_Axial_DIN0309_L9.0mm_D3.2mm_P12.70mm_Horizontal
- removed mouse-bite-2mm-slot: VAL**, Panelization:mouse-bite-2mm-slot
- added J3: from_arduino, Connector_IDC:IDC-Header_2x03_P2.54mm_Vertical, F.Cu at (138.5, 53.2)
- D2: footprint LED_THT:LED_D5.0mm -> LED_THT:LED_D5.0mm_Clear
- moved D1 6.34 mm to (139.3, 79.6), turned to 180 degrees
Routing:
- net Net-(D4-A): track 27.1 -> 0.00 mm
- net Net-(D3-GA): track 23.7 -> 0.00 mm
- net Net-(D3-BA): track 23.3 -> 0.00 mm
- net Net-(D3-RA): track 12.7 -> 0.00 mm
- net Net-(D1-RA): track 19.0 -> 7.31 mm
- net Net-(D1-GA): track 17.5 -> 6.46 mm
- net Net-(J2-Pin_7): track 10.0 -> 0.00 mm
- net Net-(J2-Pin_6): track 9.75 -> 0.00 mm
- net Net-(J2-Pin_9): track 9.27 -> 0.00 mm
- net Net-(J2-Pin_8): track 5.68 -> 0.00 mm
- net Net-(J3-Pin_2): track 6.06 -> 8.37 mm
- net Net-(J3-Pin_4): track 7.54 -> 5.98 mm
- net Net-(D1-BA): track 7.24 -> 6.34 mm
- net Net-(J3-Pin_3): track 9.24 -> 8.67 mm
Other:
- board size 48.9 x 36.5 mm -> 23.4 x 36.5 mm
- board text removed: "this side is populated"
